Commit message: remove extra elements in world and manually specify gain/amplitude for waves

File: heron_gazebo/worlds/wildlife_task.world.xacro (robot description, xacro)
@@ -7,72 +7,5 @@
     <!--Waves-->
     <xacro:include filename="$(find wave_gazebo)/world_models/ocean_waves/model.xacro"/>
-    <xacro:ocean_waves scale="2.5"/>
-    <!--wind for the wamv-->
-    <xacro:include filename="$(find vrx_gazebo)/worlds/xacros/usv_wind_plugin.xacro"/>
-    <xacro:usv_wind_gazebo direction = "270" ros_update_rate="10">
-      <wind_objs>
-        <wind_obj>
-          <name>wamv</name>
-          <link_name>wamv/base_link</link_name>
-          <coeff_vector>.5 .5 .33</coeff_vector>
-        </wind_obj>
-      </wind_objs>
-    </xacro:usv_wind_gazebo>
-    <!-- The VRX animal buoys -->
-    <include>
-      <name>crocodile_buoy</name>
-      <pose>-552 170 0 0 0 0</pose>
-      <uri>model://crocodile_buoy</uri>
-    </include>
-    <include>
-      <name>platypus_buoy</name>
-      <pose>-512 170 0 0 0 0</pose>
-      <uri>model://platypus_buoy</uri>
-    </include>
-    <include>
-      <name>turtle_buoy</name>
-      <pose>-472 170 0 0 0 0</pose>
-      <uri>model://turtle_buoy</uri>
-    </include>
-    <!-- The scoring plugin -->
-    <plugin name="wildlife_scoring_plugin"
-            filename="libwildlife_scoring_plugin.so">
-      <!-- Common parameters -->
-      <vehicle>wamv</vehicle>
-      <task_name>wildlife</task_name>
-      <initial_state_duration>10</initial_state_duration>
-      <ready_state_duration>10</ready_state_duration>
-      <running_state_duration>300</running_state_duration>
-      <collision_buffer>10</collision_buffer>
-      <release_joints>
-        <joint>
-          <name>wamv_external_pivot_joint</name>
-        </joint>
-        <joint>
-          <name>wamv_external_riser</name>
-        </joint>
-      </release_joints>
-      <!-- wildlife specific parameters -->
-      <buoys>
-        <buoy>
-          <model_name>crocodile_buoy</model_name>
-          <link_name>link</link_name>
-          <goal>avoid</goal>
-        </buoy>
-        <buoy>
-          <model_name>platypus_buoy</model_name>
-          <link_name>link</link_name>
-          <goal>circumnavigate_clockwise</goal>
-        </buoy>
-        <buoy>
-          <model_name>turtle_buoy</model_name>
-          <link_name>link</link_name>
-          <goal>circumnavigate_counterclockwise</goal>
-        </buoy>
-      </buoys>
-      <engagement_distance>10.0</engagement_distance>
-      <time_bonus>30.0</time_bonus>
-      <animals_topic>/vrx/wildlife/animals/poses</animals_topic>
-    </plugin>
+    <xacro:ocean_waves gain="0.1" scale="1.5"/>
   </world>
 </sdf>
